Commit message: refactor(boat_description): phase P3 — REP-105 + Autoware TF naming
Add livox_link, oculus_link, ping360_link, ping1d_link, sonoptix_link
per workspace conventions spec §2.2.

Legacy aliases (body, oculus, livox_frame) preserved for old bag
compatibility.

- boat_description/urdf/boat.urdf: 5 new links + 5 fixed joints
- boat_description/CHANGELOG.md: P3 entry

Verification:
- XML parse PASS
- colcon build PASS
- robot_state_publisher publishes new frames to /tf_static

File: boat_description/urdf/boat.urdf (robot description, URDF)
Before this commit: robot boat, 6 links, 5 joints
Links:
- added link livox_link
- added link oculus_link
- added link ping1d_link
- added link ping360_link
- added link sonoptix_link
Joints:
- added joint base_to_livox_link: type fixed, parent base_link, child livox_link, origin xyz=0 0 0 rpy=0 0 0
- added joint sonar_to_oculus_link: type fixed, parent sonar_link, child oculus_link, origin xyz=0 0 0 rpy=0 0 0
- added joint sonar_to_ping1d_link: type fixed, parent sonar_link, child ping1d_link, origin xyz=0 0 0 rpy=0 0 0
- added joint sonar_to_ping360_link: type fixed, parent sonar_link, child ping360_link, origin xyz=0 0 0 rpy=0 0 0
- added joint sonar_to_sonoptix_link: type fixed, parent sonar_link, child sonoptix_link, origin xyz=0 0 0 rpy=0 0 0
